Commit message: add imu
Signed-off-by: Jvle <keke.oerv@isrc.iscas.ac.cn>

File: src/my_robot_description/urdf/robot.xacro (robot description, xacro)
@@ -18,4 +18,5 @@
   <!-- Sensor -->
   <xacro:lidar_sensor name="laser" parent="base_link" xyz="0 0 0.1" rpy="0 0 0"/>
+  <xacro:imu_sensor name="imu" parent="base_link" xyz="0.05 0.05 0.05" rpy="0 0 0"/>
   <!-- Gazebo diff drive plugin -->
   <xacro:gazebo_control_plugin

File: src/my_robot_description/urdf/sensors.xacro (robot description, xacro)
@@ -40,5 +40,5 @@
         <topic>scan</topic>
         <gz_frame_id>${name}_link</gz_frame_id>
-        <lidar>
+        <ray>
           <scan>
             <horizontal>
@@ -58,5 +58,42 @@
             <max>12</max>
           </range>
-        </lidar>
+        </ray>
+      </sensor>
+    </gazebo>
+  </xacro:macro>
+  <xacro:macro name="imu_sensor" params="
+        name
+        parent
+        xyz
+        rpy">
+    <link name="${name}_link">
+      <visual>
+          <origin xyz="${xyz}" rpy="${rpy}"/>
+          <geometry>
+              <box size="0.01 0.01 0.01"/>
+          </geometry>
+          <material name="${name}_material">
+              <color rgba="0.63 0.63 0.63 1.0"/>
+          </material>
+      </visual>
+      <inertial>
+        <mass value="0.01"/>
+        <inertia
+          ixx="0.0001" ixy="0.0" ixz="0.0"
+          iyy="0.0001" iyz="0.0" izz="0.0001"/>
+      </inertial>
+    </link>
+    <joint name="${name}_joint" type="fixed">
+      <parent link="${parent}"/>
+      <child  link="${name}_link"/>
+      <origin xyz="${xyz}" rpy="${rpy}"/>
+    </joint>
+    <gazebo reference="${name}_link">
+      <sensor name="${name}_link" type="imu">
+          <topic>imu</topic>
+          <update_rate>1</update_rate>
+          <always_on>1</always_on>
+          <visualize>true</visualize>
+          <gz_frame_id>${name}_link</gz_frame_id>
       </sensor>
     </gazebo>

Commit message: add depth camera
Signed-off-by: Jvle <keke.oerv@isrc.iscas.ac.cn>

File: src/my_robot_description/urdf/robot.xacro (robot description, xacro)
@@ -19,4 +19,9 @@
   <xacro:lidar_sensor name="laser" parent="base_link" xyz="0 0 0.1" rpy="0 0 0"/>
   <xacro:imu_sensor name="imu" parent="base_link" xyz="0.05 0.05 0.05" rpy="0 0 0"/>
+  <xacro:depth_camera
+    name="camera"
+    parent="base_link"
+    xyz="0.2 0 0.1"
+    rpy="0 0 0"/>
   <!-- Gazebo diff drive plugin -->
   <xacro:gazebo_control_plugin

File: src/my_robot_description/urdf/sensors.xacro (robot description, xacro)
@@ -99,3 +99,62 @@
     </gazebo>
   </xacro:macro>
+  <xacro:macro name="depth_camera" params="
+      name
+      parent
+      xyz
+      rpy">
+    <link name="${name}_link">
+      <inertial>
+        <mass value="0.05"/>
+        <inertia
+          ixx="0.0001" ixy="0.0" ixz="0.0"
+          iyy="0.0001" iyz="0.0" izz="0.0001"/>
+      </inertial>
+      <visual>
+        <geometry>
+          <box size="0.05 0.4 0.04"/>
+        </geometry>
+        <material name="CameraGray">
+          <color rgba="0.5 0.5 0.5 1.0"/>
+        </material>
+      </visual>
+      <collision>
+        <geometry>
+          <box size="0.05 0.4 0.04" />
+        </geometry>
+      </collision>
+    </link>
+    <joint name="${name}_joint" type="fixed">
+      <parent link="${parent}"/>
+      <child  link="${name}_link"/>
+      <origin xyz="${xyz}" rpy="${rpy}"/>
+    </joint>
+    <gazebo reference="${name}_link">
+      <sensor name="${name}_link" type="rgbd_camera">
+          <always_on>true</always_on>
+          <visualize>true</visualize>
+          <update_rate>100</update_rate>
+          <topic>camera</topic>
+          <gz_frame_id>${name}_link</gz_frame_id>
+          <camera name="${name}_link">
+              <camera_info_topic>camera/camera_info</camera_info_topic>
+              <horizontal_fov>1.3962634</horizontal_fov>
+              <image>
+              <width>800</width>
+              <height>600</height>
+              <format>R8G8B8</format>
+              </image>
+              <clip>
+              <near>0.1</near>
+              <far>100</far>
+              </clip>
+              <noise>
+              <type>gaussian</type>
+              <mean>0</mean>
+              <stddev>0.007</stddev>
+              </noise>
+          </camera>
+      </sensor>
+    </gazebo>
+  </xacro:macro>
 </robot>
