Commit message: fix car's forward speed
Signed-off-by: Jvle <keke.oerv@isrc.iscas.ac.cn>

File: src/my_robot_description/urdf/base.xacro (robot description, xacro)
@@ -33,5 +33,5 @@
     </link>
     <joint name="joint_name" type="fixed">
-      <origin xyz="0 0 ${base_size_z / 2}" rpy="0 0 0"/>
+      <origin xyz="0 0 ${base_size_z + 0.05}" rpy="0 0 0"/>
       <parent link="base_footprint"/>
       <child link="base_link"/>

File: src/my_robot_description/urdf/plugins/gazebo_control_plugin.xacro (robot description, xacro)
@@ -18,5 +18,4 @@
         <wheel_separation>${wheel_separation}</wheel_separation>
         <wheel_radius>${wheel_radius}</wheel_radius>
-        <max_linear_acceleration>${max_accel}</max_linear_acceleration>
         <!-- ROS 接口（通过 ros_gz_bridge 使用） -->
         <topic>${cmd_vel_topic}</topic>
