Commit message: init nav2 for micro-ros-car
Signed-off-by: Jvle <keke.oerv@isrc.iscas.ac.cn>

File: src/robot_pkg/urdf/robot.urdf (robot description, URDF)
Before this commit: robot my_robot, 3 links, 2 joints
Links:
- removed link link1
- removed link link2
- added link base_footprint
- added link laser_link; visual cylinder length=0.02 radius=0.02
- link base_link: geometry visual cylinder length=0.12 radius=0.10
Joints:
- removed joint joint1
- removed joint joint2
- added joint base_joint: type fixed, parent base_footprint, child base_link, origin xyz=0.0 0.0 0.076 rpy=0 0 0
- added joint laser_joint: type fixed, parent base_link, child laser_link, origin xyz=0 0 0.075 rpy=0 0 0

Commit message: update repo
Signed-off-by: Jvle <keke.oerv@isrc.iscas.ac.cn>

File: src/robot_pkg/urdf/robot.urdf (robot description, URDF)
Before this commit: robot fishbot, 3 links, 2 joints
Links:
- link base_link: geometry visual cylinder length=0.12 radius=0.225
